Commit message: feat/update rover model; rename megarover3 to zestyrover and update launch parameters

File: description/urdf/zestyrover/zestyrover.urdf (robot description, URDF)
Before this commit: robot megarover3, 9 links, 8 joints
Links:
- link base_link: geometry visual mesh filename=package://description/meshes/zestyrover/zestyrover.stl
